Commit message: adding motor controller test joint

File: robot_urdf/urdf/robot4.xacro (robot description, xacro)
@@ -144,3 +144,25 @@
 	    <limit effort="1000.0" velocity="0.2"/>
 	 </joint>
+  <!-- Prove per creare un nuovo link-->
+  <link name='test_link'>
+    <visual>
+      <origin xyz="0 0 0" rpy="0 0 0"/>   <!-- frame centrato con il box -->
+      <geometry>
+        <box size="0.1 0.1 0.1"/>
+      </geometry>
+      <material name="green"/>
+    </visual>
+    <collision name="collision_test_link">
+      <origin xyz="0 0 0" rpy="0 0 0"/>
+      <geometry>
+        <box size="0.1 0.1 0.1"/>
+      </geometry>
+    </collision>
+  </link>
+  <joint name="test_joint" type="continuous">
+    <axis xyz="0 0 1"/>
+    <parent link="link_chassis"/>
+    <child link="test_link"/>
+    <origin xyz="0 0 0.2" rpy="0 0 0"/>
+  </joint>
 </robot>
